File: Hardware/Electronics/OpenPixelPoi/OpenPixelPoi.kicad_sch (KiCad schematic)
At the start: 54 parts, among them J4 Conn_01x04, J5 Conn_01x04, J6 USB_C_Receptacle_USB2.0_16P, J7 Conn_01x04, SW1 SW_Push, SW2 SW_Push, SW3 SW_Push, U1 USBLC6-2P6, U10 SN74LV1T34DBV, U2 MCP73831-2-OT, U3 ESP32-C3-MINI-1-N4, U4 XC6210B332MR, U5 TPS61023DRLR, U6 SN74LV1T34DBV, U7 FPC-0.5HF-8PWBH10, U8 FPC-0.5HF-8PWBH10, U9 FPC-0.5HF-8PWBH10

Commit message: Final pcb tweaks before large order
Parts:
- SW1, SW2: LCSC C231329 -> C19270949
